File: desgin/nixie_alarm_main_board/nixie_alarm_main_board.kicad_pcb (KiCad board)
At the start: 2 copper layers, 144.3 x 59 mm, 102 parts, among them IC1 LM3488MM, IC2 HV5530PG-G, IC3 TPS563219ADDFR, IC4 HV5530PG-G, IC6 CD40109BQNSRQ1, IC7 AP7363-33D-13, IC8 MCP4018T-502E_LT, J1 DCPLUG 2x6.4mm 2A, J2 JST XH 2.54 3 pin, J3 USB_C_Receptacle_USB2.0_16P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

Commit message: board v1
Parts:
- C10, C11, C12, C13, D2, IC1, Q9, R10, R12, R13, R14: moved to B.Cu
- C6, C7: moved to F.Cu
- moved LS1 41.6 mm to (89.6, 28.8), turned to 0 degrees
- moved Q1 29.9 mm to (97.8, 30.7), turned to 180 degrees
- moved D2 29.6 mm to (214.6, 67.0), turned to 180 degrees
- moved R35 24.9 mm to (97.8, 33.9), turned to 180 degrees
- moved C13 23.9 mm to (189.7, 56.5), turned to 0 degrees
- moved R14 20.1 mm to (194.0, 56.5), turned to 0 degrees
- moved R43 15.8 mm to (214.3, 54.9), turned to 180 degrees
- moved R42 15.8 mm to (214.3, 52.8), turned to 180 degrees
- moved C23 15.5 mm to (116.8, 57.8)
- moved R10 12.6 mm to (209.2, 56.1), turned to 180 degrees
- moved C12 10.9 mm to (208.9, 58.5), turned to 180 degrees
- moved R15 10.5 mm to (116.9, 51.8)
- moved C6 10.5 mm to (146.0, 29.9), turned to -90 degrees
- moved IC8 10.4 mm to (214.3, 57.6)
- moved R11 9.66 mm to (214.3, 60.6), turned to 0 degrees
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Connections:
- IC6 pad 7: Net-(IC6-ENABLE_B) -> +3.3V
- IC6 pad 9: Net-(IC6-ENABLE_B) -> +3.3V
- U1 pad 10: NX_DOT_5 -> BUZZER
- U1 pad 11: NX_DOT_6 -> HV_FB
- U1 pad 12: DPOT_SDA -> NX_DOT_3
- U1 pad 15: ENC_SW -> NX_BL
- U1 pad 17: DPOT_SCL -> NX_DATA_INPUT
- U1 pad 18: NX_BL -> NX_LE
- U1 pad 20: NX_LE -> NX_DOT_4
- U1 pad 21: NX_DOT_1 -> ENC_SW
- U1 pad 22: NX_DOT_2 -> NX_DOT_5
- U1 pad 23: unconnected-(U1-IO21-Pad23) -> NX_DOT_6
- U1 pad 24: unconnected-(U1-IO47-Pad24) -> DPOT_SCL
- U1 pad 25: unconnected-(U1-IO48-Pad25) -> DPOT_SDA
- U1 pad 31: unconnected-(U1-IO38-Pad31) -> ENC_B
- U1 pad 38: LED_DATA -> ENC_A
- U1 pad 39: HV_FB -> LED_DATA
- U1 pad 4: ENC_A -> NX_DOT_1
- U1 pad 5: ENC_B -> unconnected-(U1-IO5-Pad5)
- U1 pad 6: BUZZER -> unconnected-(U1-IO6-Pad6)
- U1 pad 7: NX_DATA_INPUT -> unconnected-(U1-IO7-Pad7)
- U1 pad 8: NX_DOT_3 -> unconnected-(U1-IO15-Pad8)
- U1 pad 9: NX_DOT_4 -> NX_DOT_2
Routing:
- net +3.3V: track 137.6 -> 282.1 mm, vias 6 -> 3
- net DPOT_SCL: track 9.53 -> 129.8 mm, vias 0 -> 2
- net DPOT_SDA: track 9.00 -> 126.2 mm, vias 0 -> 2
- net NX_DOT_6: track 2.07 -> 110.4 mm, vias 0 -> 1
- net NX_DOT_5: track 2.06 -> 90.5 mm, vias 0 -> 1
- net NX_CLK: track 5.13 -> 83.8 mm, vias 2 -> 4
- net NX_LE: track 5.05 -> 82.8 mm, vias 2 -> 4
- net NX_BL: track 4.97 -> 71.3 mm, vias 2 -> 4
- net NX_DATA_INPUT: track 7.18 -> 72.3 mm, vias 3 -> 4
- net NX_DOT_4: track 3.85 -> 63.1 mm
- net ENC_SW: track 1.91 -> 48.1 mm, vias 0 -> 2
- net NX_DOT_3: track 3.68 -> 48.7 mm
- net LED_DATA: track 2.28 -> 46.6 mm, vias 1 -> 0
- net +12V: track 243.9 -> 284.1 mm, vias 10 -> 18
- net HV_FB: track 4.60 -> 30.2 mm, vias 1 -> 2
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- added copper zone on B.Cu, net +12V
- added copper zone on F.Cu, net +12V

Commit message: ground
Parts:
- added REF**: MountingHole_3.2mm_M3_Pad_Via, MountingHole:MountingHole_3.2mm_M3_Pad_Via, F.Cu at (220.3, 69.6)
- added REF**: MountingHole_3.2mm_M3_Pad_Via, MountingHole:MountingHole_3.2mm_M3_Pad_Via, F.Cu at (85.1, 120.6)
- added REF**: MountingHole_3.2mm_M3_Pad_Via, MountingHole:MountingHole_3.2mm_M3_Pad_Via, F.Cu at (85.0, 69.6)
- added REF**: MountingHole_3.2mm_M3_Pad_Via, MountingHole:MountingHole_3.2mm_M3_Pad_Via, F.Cu at (220.3, 120.5)
- moved C8 48.1 mm to (178.0, 69.9)
- moved R44 46.9 mm to (203.7, 103.2)
- moved U1 46.8 mm to (93.5, 107.3)
- moved C14 46.8 mm to (159.4, 121.2)
- moved C15 46.8 mm to (146.7, 121.2)
- moved C16 46.8 mm to (213.7, 100.4)
- moved C20 46.8 mm to (167.4, 105.7)
- moved C22 46.8 mm to (173.8, 104.7)
- moved C24 46.8 mm to (137.0, 119.2)
- moved C25 46.8 mm to (111.2, 112.7)
- moved C28 46.8 mm to (89.7, 95.2)
- moved IC1 46.8 mm to (207.8, 108.4)
- moved IC2 46.8 mm to (128.6, 76.4)
- moved R12 46.8 mm to (219.2, 110.4)
- moved R13 46.8 mm to (207.8, 103.2)
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Routing:
- net GND: track 6.15 -> 19.3 mm, vias 0 -> 72
- net +5V: track 96.3 -> 101.3 mm
- net +12V: track 284.1 -> 279.9 mm
- net Net-(IC3-SW): track 9.25 -> 11.9 mm
- net Net-(D2-A): track 35.0 -> 36.2 mm
- net NX_DOT_6: track 110.4 -> 109.6 mm
- net DPOT_SCL: track 129.8 -> 130.3 mm
- added copper zone on B.Cu, net GND
- added copper zone on F.Cu, net GND
Other:
- board size 144.3 x 59 mm -> 144.4 x 59.1 mm
- board text removed: "FRONT"

Commit message: new layout
Parts:
- removed Q9: TPH5200FNH,L1Q, Package_SO:SO-8_3.9x4.9mm_P1.27mm
- removed the REF** at (220.3, 69.6)
- removed the REF** at (85.1, 120.6)
- removed the REF** at (85.0, 69.6)
- removed the REF** at (220.3, 120.5)
- added Q8: TPH5200FNH,L1Q, SamacSys_Parts:TPHR6503PL1LQ, F.Cu at (217.8, 134.8)
- added REF**: MountingHole_3.2mm_M3_Pad_Via, MountingHole:MountingHole_3.2mm_M3_Pad_Via, F.Cu at (217.7, 115.4)
- added REF**: MountingHole_3.2mm_M3_Pad_Via, MountingHole:MountingHole_3.2mm_M3_Pad_Via, F.Cu at (88.2, 115.7)
- added REF**: MountingHole_3.2mm_M3_Pad_Via, MountingHole:MountingHole_3.2mm_M3_Pad_Via, F.Cu at (217.8, 71.2)
- added REF**: MountingHole_3.2mm_M3_Pad_Via, MountingHole:MountingHole_3.2mm_M3_Pad_Via, F.Cu at (88.1, 71.1)
- C26, C27, IC3, IC6, IC7, R1, R2, R5: moved to F.Cu
- moved LS1 125.2 mm to (215.6, 106.0)
- moved C21 74.3 mm to (245.8, 140.2)
- moved C22 70.1 mm to (226.4, 150.9)
- moved C13 56.8 mm to (244.7, 129.3)
- moved R14 56.8 mm to (249.0, 129.3)
- moved R21 56.6 mm to (72.5, 96.1)
- moved R15 49.6 mm to (72.6, 106.5)
- moved C19 48.3 mm to (70.2, 118.9)
- moved C20 47.9 mm to (204.3, 136.2)
- moved C23 47.9 mm to (74.5, 113.5)
- moved J2 46.9 mm to (86.5, 103.5), turned to -90 degrees
- moved C18 46.5 mm to (67.3, 101.8)
- moved C3 45.3 mm to (139.6, 149.7)
- moved R1 38.6 mm to (102.4, 110.2), turned to 0 degrees
- moved R2 38.5 mm to (102.4, 108.0), turned to 180 degrees
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Routing:
- net +3.3V: track 282.5 -> 31.3 mm, vias 3 -> 0
- net DPOT_SCL: track 130.3 -> 0.00 mm, vias 2 -> 0
- net DPOT_SDA: track 126.2 -> 0.00 mm, vias 2 -> 0
- net NX_DOT_6: track 109.6 -> 0.00 mm, vias 1 -> 0
- net +12V: track 279.9 -> 177.8 mm, vias 18 -> 2
- net NX_DOT_5: track 90.5 -> 0.00 mm, vias 1 -> 0
- net ENC_B: track 75.0 -> 2.62 mm, vias 2 -> 0
- net NX_CLK: track 83.8 -> 12.1 mm, vias 4 -> 2
- net NX_LE: track 82.8 -> 12.4 mm, vias 4 -> 2
- net HV: track 152.0 -> 82.8 mm
- net NX_DOT_4: track 63.1 -> 0.00 mm, vias 1 -> 0
- net ENC_A: track 64.6 -> 2.73 mm, vias 2 -> 0
- net NX_DATA_INPUT: track 72.3 -> 12.3 mm, vias 4 -> 2
- net NX_BL: track 71.3 -> 12.0 mm, vias 4 -> 2
- net NX_DOT_3: track 48.7 -> 0.21 mm, vias 1 -> 0
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- removed copper zone on B.Cu, net +12V
- removed copper zone on F.Cu, net +12V
- removed copper zone on B.Cu, net GND
- removed copper zone on F.Cu, net GND
Other:
- board size 144.4 x 59.1 mm -> 138.2 x 53 mm

Commit message: hv section
Parts:
- C11, C12, C5, D2, IC1, IC8, R10, R12, R13, R42, R43: moved to F.Cu
- moved C5 64.5 mm to (102.4, 103.7), turned to 180 degrees
- moved C3 55.9 mm to (102.5, 107.9), turned to 90 degrees
- moved D2 49.6 mm to (188.8, 103.9), turned to 0 degrees
- moved IC1 41.6 mm to (205.3, 103.5)
- moved C11 37.6 mm to (208.4, 107.2)
- moved Q8 36.0 mm to (197.3, 105.1), turned to 90 degrees
- moved R44 35.1 mm to (199.9, 103.8)
- moved C12 35.0 mm to (210.7, 103.9)
- moved R13 34.1 mm to (204.1, 106.7)
- moved R10 29.4 mm to (215.9, 103.9), turned to 0 degrees
- moved R11 26.0 mm to (212.2, 115.3), turned to -90 degrees
- moved R43 26.0 mm to (212.2, 109.1), turned to -90 degrees
- moved R12 25.1 mm to (212.8, 114.9), turned to -90 degrees
- moved IC8 22.2 mm to (215.5, 109.5), turned to 180 degrees
- moved R42 20.4 mm to (218.8, 109.1), turned to -90 degrees
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Routing:
- net HV: track 82.8 -> 114.4 mm, vias 0 -> 1
- net Net-(IC1-FB): track 0.28 -> 18.8 mm, vias 0 -> 2
- net Net-(D2-A): track 0.00 -> 15.9 mm, vias 0 -> 1
- net +12V: track 177.8 -> 192.6 mm
- net +3.3V: track 31.3 -> 40.2 mm
- net Net-(IC8-A): track 0.00 -> 7.35 mm, vias 0 -> 1
- net Net-(IC1-COMP): track 0.00 -> 6.39 mm
- net Net-(Q8-S_1): track 0.77 -> 6.43 mm
- net +5V: track 96.5 -> 100.4 mm
- net Net-(IC1-ISEN): track 0.00 -> 3.32 mm
- net Net-(IC1-DR): track 0.00 -> 3.01 mm
- net DPOT_SCL: track 0.00 -> 2.76 mm
- net DPOT_SDA: track 0.00 -> 2.61 mm
- net Net-(IC1-FA/SYNC/SD): track 0.00 -> 2.21 mm, vias 0 -> 1
- net USB_D+: track 37.4 -> 38.6 mm
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