File: desgin/nixie_alarm_main_board/nixie_alarm_main_board.kicad_pcb (KiCad board)
At the start: 2 copper layers, 138.2 x 53 mm, 106 parts, among them IC1 LM3488MM, IC2 HV5530PG-G, IC3 TPS563219ADDFR, IC4 HV5530PG-G, IC6 CD40109BQNSRQ1, IC7 AP7363-33D-13, IC8 MCP4018T-502E_LT, J1 DCPLUG 2x6.4mm 2A, J2 JST XH 2.54 3 pin, J3 USB_C_Receptacle_USB2.0_16P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

Commit message: new board v1
Parts:
- removed C23: 100nF 25V, Capacitor_SMD:C_0805_2012Metric_Pad1.18x1.45mm_HandSolder
- C16, C17, C24, C25, C28, R3, R4: moved to F.Cu
- J1: value DCPLUG 2x6.4mm 2A -> PJ-094H-SMT-TR; footprint SamacSys_Parts:DCJ20005AK1A -> SamacSys_Parts:PJ094HSMTTR
- J2: footprint Connector_JST:JST_XH_B3B-XH-A_1x03_P2.50mm_Vertical -> Connector_JST:JST_XH_S3B-XH-A-1_1x03_P2.50mm_Horizontal
- moved Q1 148.5 mm to (218.3, 97.8), turned to 0 degrees
- moved R35 138.3 mm to (215.1, 97.8), turned to -90 degrees
- moved C21 88.9 mm to (166.2, 100.8), turned to 180 degrees
- moved C22 72.9 mm to (172.6, 101.8), turned to 90 degrees
- moved C24 62.1 mm to (95.4, 105.8), turned to 90 degrees
- moved R21 57.3 mm to (129.0, 86.7), turned to -90 degrees
- moved R14 56.7 mm to (199.5, 101.7), turned to 180 degrees
- moved C28 55.5 mm to (120.5, 112.7), turned to 0 degrees
- moved R15 53.2 mm to (122.3, 87.7), turned to 180 degrees
- moved C13 51.7 mm to (199.4, 104.2)
- moved C19 45.7 mm to (115.3, 111.2)
- moved C18 45.7 mm to (112.0, 111.2)
- moved C20 43.5 mm to (179.0, 100.8), turned to 0 degrees
- moved R16 43.1 mm to (122.5, 90.4), turned to 0 degrees
- moved C10 33.0 mm to (206.3, 105.8)
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Connections:
- U1 pad 10: BUZZER -> NX_DOT_2
- U1 pad 15: NX_BL -> NX_LE
- U1 pad 17: NX_DATA_INPUT -> NX_CLK
- U1 pad 18: NX_LE -> NX_DATA_INPUT
- U1 pad 19: NX_CLK -> NX_BL
- U1 pad 21: ENC_SW -> NX_DOT_5
- U1 pad 22: NX_DOT_5 -> BUZZER
- U1 pad 31: ENC_B -> ENC_SW
- U1 pad 38: ENC_A -> ENC_B
- U1 pad 39: LED_DATA -> ENC_A
- U1 pad 4: NX_DOT_1 -> LED_DATA
- U1 pad 5: unconnected-(U1-IO5-Pad5) -> NX_DOT_1
- U1 pad 9: NX_DOT_2 -> unconnected-(U1-IO16-Pad9)
Routing:
- net +3.3V: track 40.2 -> 285.7 mm, vias 0 -> 7
- net DPOT_SCL: track 2.76 -> 106.2 mm, vias 0 -> 3
- net NX_DOT_6: track 0.00 -> 101.7 mm, vias 0 -> 1
- net DPOT_SDA: track 2.61 -> 102.4 mm, vias 0 -> 3
- net BUZZER: track 0.00 -> 99.8 mm, vias 0 -> 2
- net +12V: track 192.6 -> 289.2 mm, vias 2 -> 6
- net HV: track 114.4 -> 201.2 mm, vias 1 -> 2
- net NX_DOT_5: track 0.00 -> 74.3 mm, vias 0 -> 1
- net NX_BL: track 12.0 -> 61.4 mm, vias 2 -> 5
- net NX_DATA_INPUT: track 12.3 -> 59.0 mm, vias 2 -> 5
- net NX_LE: track 12.4 -> 58.3 mm, vias 2 -> 3
- net NX_DOT_4: track 0.00 -> 43.3 mm, vias 0 -> 1
- net NX_DOT_3: track 0.21 -> 42.5 mm, vias 0 -> 1
- net NX_CLK: track 12.1 -> 53.4 mm, vias 2 -> 3
- net NX_DOT_1: track 0.00 -> 37.6 mm, vias 0 -> 3
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- added copper zone on B.Cu, net GND
- added copper zone on F.Cu, net GND
Other:
- outline, holes or cut-outs redrawn

Commit message: elements sings fixed
Parts:
- moved R11 2.00 mm to (212.2, 113.3)
- moved R22 1.70 mm to (107.0, 92.9)
- moved C25 0.72 mm to (104.8, 114.2)
- moved R23 0.70 mm to (101.6, 92.9)
- moved C26 0.55 mm to (106.5, 110.2)
- moved C17 0.45 mm to (108.2, 114.2)
- moved R5 0.35 mm to (106.7, 103.9)
- moved C14 0.16 mm to (159.8, 113.8)
- moved R16 0.15 mm to (122.3, 90.4)
- moved C15 0.15 mm to (147.8, 113.8)
- moved R14 0.05 mm to (199.4, 101.7)
Routing:
- net GND: track 30.9 -> 35.7 mm, vias 39 -> 47
- net +3.3V: track 285.7 -> 282.8 mm
- net DPOT_SCL: track 106.2 -> 108.7 mm
- net DPOT_SDA: track 102.4 -> 104.3 mm
- net Net-(N2-Padu): track 10.4 -> 8.68 mm
- net Net-(N1-Padu): track 3.37 -> 4.07 mm
- net Net-(D2-A): track 15.6 -> 15.0 mm
- net HV: track 201.2 -> 201.9 mm
- net Net-(N3-Padu): track 3.18 -> 3.85 mm
- net Net-(IC3-SW): track 24.7 -> 24.1 mm

Commit message: add more detalis
Parts:
- added 12V: TestPoint_Pad_D1.5mm, TestPoint:TestPoint_Pad_D1.5mm, F.Cu at (104.0, 120.2)
- added 3.3V: TestPoint_Pad_D1.5mm, TestPoint:TestPoint_Pad_D1.5mm, F.Cu at (96.8, 120.2)
- added 5V: TestPoint_Pad_D1.5mm, TestPoint:TestPoint_Pad_D1.5mm, F.Cu at (100.5, 120.2)
- added GND: TestPoint_Pad_D1.5mm, TestPoint:TestPoint_Pad_D1.5mm, F.Cu at (111.0, 120.2)
- added HV: TestPoint_Pad_D1.5mm, TestPoint:TestPoint_Pad_D1.5mm, F.Cu at (107.5, 120.2)
- added J4: JST XH 2.54 3 pin, Connector_JST:JST_EH_S2B-EH_1x02_P2.50mm_Horizontal, B.Cu at (169.8, 80.4)
- moved REF** 142.4 mm to (220.9, 122.4), turned to 180 degrees
- moved REF** 137.7 mm to (220.8, 77.9), turned to 180 degrees
- moved J2 136.6 mm to (221.7, 84.4), turned to 180 degrees
- moved REF** 136.5 mm to (91.2, 122.4), turned to 180 degrees
- moved REF** 132.4 mm to (91.1, 77.9), turned to 180 degrees
- moved R42 130.9 mm to (90.2, 84.4), turned to 90 degrees
- moved Q1 127.6 mm to (90.8, 95.7), turned to 180 degrees
- moved R29 126.6 mm to (217.8, 93.8), turned to -90 degrees
- moved IC8 124.6 mm to (93.5, 84.0), turned to 0 degrees
- moved R3 124.5 mm to (213.9, 78.2), turned to 0 degrees
- moved R10 124.4 mm to (92.7, 89.8), turned to 180 degrees
- moved C16 123.6 mm to (93.5, 86.9), turned to 180 degrees
- moved LS1 123.4 mm to (93.5, 87.4), turned to 180 degrees
- moved R12 122.1 mm to (96.2, 78.6), turned to 90 degrees
- moved R41 121.3 mm to (94.0, 93.9), turned to 90 degrees
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Routing:
- net +5V: track 111.0 -> 267.2 mm, vias 5 -> 6
- net +3.3V: track 282.8 -> 322.0 mm
- net +12V: track 288.7 -> 322.0 mm, vias 6 -> 7
- net HV: track 201.9 -> 229.7 mm, vias 2 -> 3
- net DEBUG_UART_RX: track 0.00 -> 20.3 mm
- net DEBUG_UART_TX: track 0.00 -> 14.2 mm
- net ENC_A: track 16.0 -> 17.3 mm
- net ENC_B: track 30.6 -> 31.8 mm
- net NX_DOT_6: track 101.7 -> 100.9 mm
- net GND: vias 47 -> 53
Other:
- outline, holes or cut-outs redrawn
- board text added: "5V"
- board text added: "GND"
- board text added: "HV Danger"
- board text added: "IN"
- board text added: "Nixie alarm clock"
- board text added: "Paderewski"
- board text added: "RX"
- board text added: "TX"

Commit message: copper border
Parts:
- removed J4: JST XH 2.54 3 pin, Connector_JST:JST_EH_S2B-EH_1x02_P2.50mm_Horizontal
- added J5: Goldpin 3pin, Connector_PinHeader_2.54mm:PinHeader_1x03_P2.54mm_Horizontal, B.Cu at (171.1, 83.8)
- moved R20 3.04 mm to (160.9, 79.8)
- moved C15 3.03 mm to (161.3, 76.7)
Connections:
- U1 pad 38: ENC_B -> ENC_A
- U1 pad 39: ENC_A -> ENC_B
Routing:
- net (no net): track 0.00 -> 801.8 mm
- net DEBUG_UART_RX: track 20.3 -> 6.99 mm
- net DEBUG_UART_TX: track 14.2 -> 3.63 mm
- net +5V: track 267.2 -> 269.5 mm
- net +12V: track 322.0 -> 324.1 mm
- net ENC_SW: track 18.7 -> 20.5 mm
- net ENC_B: track 31.8 -> 30.0 mm
- net NX_DOT_3: track 42.1 -> 42.8 mm
- net +3.3V: track 322.0 -> 321.8 mm, vias 7 -> 6
- net GND: vias 53 -> 56
Other:
- board size 138.2 x 53 mm -> 138.3 x 52.9 mm

Commit message: little fixes
Parts:
- moved R31 0.19 mm to (116.4, 97.6)

Commit message: little fixes
Parts:
- L1: value 2.2uH 9.2A -> 2.2uH 9.7A; footprint SamacSys_Parts:XAL5030222MEC -> SamacSys_Parts:SRP5030CA4R7M
- moved L1 0.37 mm to (203.3, 94.0), turned to 90 degrees
- turned R34 to -90 degrees
Routing:
- net +5V: track 269.2 -> 273.3 mm
- net NX_DOT_2: track 10.5 -> 8.85 mm
- net Net-(IC3-SW): track 24.1 -> 25.3 mm, vias 1 -> 2
- net +3.3V: track 321.8 -> 322.8 mm, vias 6 -> 7
- net Net-(Q7-G): track 3.56 -> 2.73 mm
- net NX_DOT_6: track 100.9 -> 101.7 mm
