File: desgin/nixie_alarm_main_board/buzzer.kicad_sch (KiCad schematic)
At the start: 1 part

Commit message: filter caps
Parts:
- removed BZ1: Buzzer, Buzzer_Beeper:MagneticBuzzer_PUI_AT-0927-TT-6-R, symbol Device:Buzzer
- added C23: 100nF 25V, GRM033D70J224ME01D, symbol SamacSys_Parts:GRM033R71E101KA01J
- added LS1: CEM-1203_42_, SamacSys_Parts:CEM-1203_42_, symbol SamacSys_Parts:CEM-1203_42_
- added Q1: SSM3K35AMFV,L3F, SSM3K35AMFVL3F, symbol SamacSys_Parts:SSM3K35AMFV,L3F
- added R35: 10k, ERJUP6, symbol SamacSys_Parts:ERJ-UP6D5101V
Connections:
- net GND: now also C23.2, Q1.2 (S)
- net buzzer: now also R35.2
- new net: LS1.2 (-), Q1.3 (D)
- new net: Q1.1 (G), R35.1
- new net +3.3V: C23.1, LS1.1 (+)

Commit message: new caps footprint
Parts:
- C23: footprint GRM033D70J224ME01D -> Capacitor_SMD:C_0805_2012Metric_Pad1.18x1.45mm_HandSolder
- R35: footprint ERJUP6 -> Resistor_SMD:R_0805_2012Metric_Pad1.20x1.40mm_HandSolder
Changed lines of the file:
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@@
 			)
 		)
-		(property "Footprint" "GRM033D70J224ME01D"
+		(property "Footprint" "Capacitor_SMD:C_0805_2012Metric_Pad1.18x1.45mm_HandSolder"
 			(at 82.88 87.63 0)
 			(effects
@@
 			)
 		)
-		(property "Footprint" "ERJUP6"
+		(property "Footprint" "Resistor_SMD:R_0805_2012Metric_Pad1.20x1.40mm_HandSolder"
 			(at 122.936 0.076 0)
 			(effects

Commit message: new board v1
Parts:
- removed C23: 100nF 25V, Capacitor_SMD:C_0805_2012Metric_Pad1.18x1.45mm_HandSolder, symbol SamacSys_Parts:GRM033R71E101KA01J
Changed lines of the file:
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@@
 	(generator_version "8.0")
 	(paper "A4")
-	(junction
-		(at 145.288 76.2)
-		(diameter 0)
-		(color 0 0 0 0)
-	)
-	(wire
-		(pts
-			(xy 179.07 76.2) (xy 145.288 76.2)
-		)
-		(stroke
-			(width 0)
-			(type default)
-		)
-	)
 	(wire
 		(pts
@@
 	(wire
 		(pts
-			(xy 179.07 78.74) (xy 179.07 76.2)
-		)
-		(stroke
-			(width 0)
-			(type default)
-		)
-	)
-	(wire
-		(pts
-			(xy 145.288 76.2) (xy 145.288 83.566)
-		)
-		(stroke
-			(width 0)
-			(type default)
-		)
-	)
-	(wire
-		(pts
 			(xy 117.094 96.266) (xy 119.126 96.266)
 		)
@@
 	(wire
 		(pts
-			(xy 145.288 73.914) (xy 145.288 76.2)
+			(xy 145.288 73.914) (xy 145.288 83.566)
 		)
 		(stroke
@@
 					(unit 1)
 				)
-			)
-		)
-	)
-	(symbol
-		(lib_id "power:GND")
-		(at 179.07 91.44 0)
-		(unit 1)
-		(exclude_from_sim no)
-		(in_bom yes)
-		(on_board yes)
-		(dnp no)
-		(fields_autoplaced yes)
-		(property "Reference" "#PWR041"
-			(at 179.07 97.79 0)
-			(effects
-				(font
-					(size 1.27 1.27)
-				)
-				(hide yes)
-			)
-		)
-		(property "Value" "GND"
-			(at 179.07 96.012 0)
-			(effects
-				(font
-					(size 1.27 1.27)
-				)
-			)
-		)
-		(property "Footprint" ""
-			(at 179.07 91.44 0)
-			(effects
-				(font
-					(size 1.27 1.27)
-				)
-				(hide yes)
-			)
-		)
-		(property "Datasheet" ""
-			(at 179.07 91.44 0)
-			(effects
-				(font
-					(size 1.27 1.27)
-				)
-				(hide yes)
-			)
-		)
-		(property "Description" "Power symbol creates a global label with name \"GND\" , ground"
-			(at 179.07 91.44 0)
-			(effects
-				(font
-					(size 1.27 1.27)
-				)
-				(hide yes)
-			)
-		)
-		(pin "1"
-		)
-		(instances
-			(project "nixie_alarm_main_board"
-				(path "/a0d555d7-39a0-4a98-b831-70d97d0aa5a1/213b4d52-76a7-4834-ad68-e02bc5e5b10b"
-					(reference "#PWR041")
-					(unit 1)
-				)
-			)
-		)
-	)
-	(symbol
-		(lib_id "SamacSys_Parts:GRM033R71E101KA01J")
-		(at 179.07 78.74 270)
-		(unit 1)
-		(exclude_from_sim no)
-		(in_bom yes)
-		(on_board yes)
-		(dnp no)
-		(property "Reference" "C23"
-			(at 184.658 83.058 90)
-			(effects
-				(font
-					(size 1.27 1.27)
-				)
-				(justify right)
-			)
-		)
-		(property "Value" "100nF 25V"
-			(at 192.532 85.09 90)
-			(effects
-				(font
-					(size 1.27 1.27)
-				)
-				(justify right)
-			)
-		)
-		(property "Footprint" "Capacitor_SMD:C_0805_2012Metric_Pad1.18x1.45mm_HandSolder"
-			(at 82.88 87.63 0)
-			(effects
-				(font
-					(size 1.27 1.27)
-				)
-				(justify left top)
-				(hide yes)
-			)
-		)
-		(property "Datasheet" "https://search.murata.co.jp/Ceramy/image/img/A01X/G101/ENG/GRM033R71E101KA01-01A.pdf"
-			(at -17.12 87.63 0)
-			(effects
-				(font
-					(size 1.27 1.27)
-				)
-				(justify left top)
-				(hide yes)
-			)
-		)
-		(property "Description" "Multilayer Ceramic Capacitors MLCC - SMD/SMT 100pF 25 volts 10%"
-			(at 179.07 78.74 0)
-			(effects
-				(font
-					(size 1.27 1.27)
-				)
-				(hide yes)
-			)
-		)
-		(property "Height" "0.5"
-			(at -217.12 87.63 0)
-			(effects
-				(font
-					(size 1.27 1.27)
-				)
-				(justify left top)
-				(hide yes)
-			)
-		)
-		(property "Mouser Part Number" "81-GRM033R71E101KA1J"
-			(at -317.12 87.63 0)
-			(effects
-				(font
-					(size 1.27 1.27)
-				)
-				(justify left top)
-				(hide yes)
-			)
-		)
-		(property "Mouser Price/Stock" "https://www.mouser.co.uk/ProductDetail/Murata-Electronics/GRM033R71E101KA01J?qs=563MOeNa05Lmru4oTW10Jw%3D%3D"
-			(at -417.12 87.63 0)
-			(effects
-				(font
-					(size 1.27 1.27)
-				)
-				(justify left top)
-				(hide yes)
-			)
-		)
-		(property "Manufacturer_Name" "Murata Electronics"
-			(at -517.12 87.63 0)
-			(effects
-				(font
-					(size 1.27 1.27)
-				)
-				(justify left top)
-				(hide yes)
-			)
-		)
-		(property "Manufacturer_Part_Number" "GRM033R71E101KA01J"
-			(at -617.12 87.63 0)
-			(effects
-				(font
-					(size 1.27 1.27)
-				)
-				(justify left top)
-				(hide yes)
-			)
-		)
-		(pin "1"
-		)
-		(pin "2"
-		)
-		(instances
-			(project "nixie_alarm_main_board"
-				(path "/a0d555d7-39a0-4a98-b831-70d97d0aa5a1/213b4d52-76a7-4834-ad68-e02bc5e5b10b"
-					(reference "C23")
-					(unit 1)
-				)

Commit message: fixes added
Parts:
- added D5: CDBUR0520, Diode_SMD:D_0603_1608Metric_Pad1.05x0.95mm_HandSolder, symbol Device:D
Connections:
- net +3.3V: now also D5.1 (K)
- net at LS1.2 (-), Q1.3 (D): now also D5.2 (A)
Other:
- moved on the sheet: LS1, Q1, R35
