File: desgin/nixie_alarm_main_board/12V_to_5V_conv.kicad_sch (KiCad schematic)
At the start: 9 parts, among them IC3 TPS563219ADDFR

Commit message: board v2
Parts:
- removed C1: 100uF 16V, CAPPM7344X310N, symbol SamacSys_Parts:TAJD107K016RNJ
- removed C3: 100nF 25V, Capacitor_SMD:C_0805_2012Metric_Pad1.18x1.45mm_HandSolder, symbol SamacSys_Parts:GRM033R71E101KA01J
- added C1, C29: 22uF 10V, Capacitor_SMD:C_0805_2012Metric_Pad1.18x1.45mm_HandSolder, symbol Device:C
- C27: value 10pF 25V -> 10nF 25V
Connections:
- net +5V: now also C1.1, C29.1
- net GND: now also C1.2, C29.2
Other:
- note removed: "Tantal"
- moved on the sheet: C26, C27, C5, IC3, L1, R1, R2
