File: desgin/nixie_alarm_main_board/12V_to_HV_conv.kicad_sch (KiCad schematic)
At the start: 22 parts, among them IC1 LM3488MM, IC8 MCP4018T-502E_LT, Q8 TPH5200FNH,L1Q

Commit message: board v2
Parts:
- removed C2: 12uF 250V, Capacitor_THT:CP_Radial_D10.0mm_P5.00mm, symbol Device:C_Polarized
- added C2, C23: 2.2uF 250 V, Capacitor_SMD:C_2220_5750Metric_Pad1.97x5.40mm_HandSolder, symbol Device:C
- added D6: 3.6V, Diode_SMD:D_0805_2012Metric_Pad1.15x1.40mm_HandSolder, symbol Device:D_Zener
- IC8: value MCP4018T-502E_LT -> MCP4018T-103E/LT
- R16: value 14.3kΩ -> 10kΩ
- R44: value 27kΩ -> 35.7kΩ
Connections:
- net GND: now also C2.2, C23.2, D6.2 (A)
- net HV_FB: now also D6.1 (K)
- net at D2.1 (K), R12.1, R5.1: now also C2.1, C23.1
Other:
- note removed: "horizontal len. 12.5mm diamiter: 10mm"
- moved on the sheet: C11, C12, C13, D2, IC1, L2, Q8, R10, R13, R14, R15, R16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
