File: desgin/nixie_alarm_main_board/LED_strip.kicad_sch (KiCad schematic)
At the start: 3 parts, among them J2 JST XH 2.54 3 pin

Commit message: board v2
Parts:
- R6: value 470Ω -> 100Ω
Changed lines of the file:
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@@
 			)
 		)
-		(property "Value" "470Ω"
+		(property "Value" "100Ω"
 			(at 160.02 100.33 0)
 			(effects
