File: desgin/nixie_alarm_main_board/nixie.kicad_sch (KiCad schematic)
At the start: 41 parts, among them IC2 HV5530PG-G, IC4 HV5530PG-G, IC6 CD40109BQNSRQ1, Q2 DMN60H080DS-13, Q3 DMN60H080DS-13, Q4 DMN60H080DS-13, Q5 DMN60H080DS-13, Q6 DMN60H080DS-13, Q7 DMN60H080DS-13

Commit message: board v2
Parts:
- R22, R23, R25, R28, R31, R33: value 27kΩ -> 35.7kΩ
Connections:
- net DATA_INPUT: now also IC6.10 (C); no longer IC6.5 (F)
- net LE: now also IC6.14 (D); no longer IC6.4 (E)
- net N1_0: now also IC2.36 (HVOUT2); no longer IC2.44 (HVOUT10)
- net N1_2: now also IC2.44 (HVOUT10); no longer IC2.36 (HVOUT2)
- net N1_3: now also IC2.43 (HVOUT9); no longer IC2.37 (HVOUT3)
- net N1_4: now also IC2.42 (HVOUT8); no longer IC2.38 (HVOUT4)
- net N1_5: now also IC2.41 (HVOUT7); no longer IC2.39 (HVOUT5)
- net N1_7: now also IC2.39 (HVOUT5); no longer IC2.41 (HVOUT7)
- net N1_8: now also IC2.38 (HVOUT4); no longer IC2.42 (HVOUT8)
- net N1_9: now also IC2.37 (HVOUT3); no longer IC2.43 (HVOUT9)
- net N2_0: now also IC2.2 (HVOUT12); no longer IC2.10 (HVOUT20)
- net N2_2: now also IC2.10 (HVOUT20); no longer IC2.2 (HVOUT12)
- net N2_3: now also IC2.9 (HVOUT19); no longer IC2.3 (HVOUT13)
- net N2_4: now also IC2.8 (HVOUT18); no longer IC2.4 (HVOUT14)
- net N2_5: now also IC2.7 (HVOUT17); no longer IC2.5 (HVOUT15)
- net N2_7: now also IC2.5 (HVOUT15); no longer IC2.7 (HVOUT17)
- net N2_8: now also IC2.4 (HVOUT14); no longer IC2.8 (HVOUT18)
- net N2_9: now also IC2.3 (HVOUT13); no longer IC2.9 (HVOUT19)
- net N3_0: now also IC2.13 (HVOUT23); no longer IC2.21 (HVOUT31)
- net N3_2: now also IC2.21 (HVOUT31); no longer IC2.13 (HVOUT23)
- net N3_3: now also IC2.20 (HVOUT30); no longer IC2.14 (HVOUT24)
- net N3_4: now also IC2.19 (HVOUT29); no longer IC2.15 (HVOUT25)
- net N3_5: now also IC2.18 (HVOUT28); no longer IC2.16 (HVOUT26)
- net N3_7: now also IC2.16 (HVOUT26); no longer IC2.18 (HVOUT28)
- net N3_8: now also IC2.15 (HVOUT25); no longer IC2.19 (HVOUT29)
- net N3_9: now also IC2.14 (HVOUT24); no longer IC2.20 (HVOUT30)
- net N4_0: now also IC4.36 (HVOUT2); no longer IC4.44 (HVOUT10)
- net N4_2: now also IC4.44 (HVOUT10); no longer IC4.36 (HVOUT2)
- net N4_3: now also IC4.43 (HVOUT9); no longer IC4.37 (HVOUT3)
- net N4_4: now also IC4.42 (HVOUT8); no longer IC4.38 (HVOUT4)
- net N4_5: now also IC4.41 (HVOUT7); no longer IC4.39 (HVOUT5)
- net N4_7: now also IC4.39 (HVOUT5); no longer IC4.41 (HVOUT7)
- net N4_8: now also IC4.38 (HVOUT4); no longer IC4.42 (HVOUT8)
- net N4_9: now also IC4.37 (HVOUT3); no longer IC4.43 (HVOUT9)
- net N5_0: now also IC4.3 (HVOUT13); no longer IC4.11 (HVOUT21)
- net N5_2: now also IC4.11 (HVOUT21); no longer IC4.3 (HVOUT13)
- net N5_3: now also IC4.10 (HVOUT20); no longer IC4.4 (HVOUT14)
- net N5_4: now also IC4.9 (HVOUT19); no longer IC4.5 (HVOUT15)
- net N5_5: now also IC4.8 (HVOUT18); no longer IC4.6 (HVOUT16)
- net N5_7: now also IC4.6 (HVOUT16); no longer IC4.8 (HVOUT18)
- net N5_8: now also IC4.5 (HVOUT15); no longer IC4.9 (HVOUT19)
- net N5_9: now also IC4.4 (HVOUT14); no longer IC4.10 (HVOUT20)
- net N6_0: now also IC4.14 (HVOUT24); no longer IC4.22 (HVOUT32)
- net N6_2: now also IC4.22 (HVOUT32); no longer IC4.14 (HVOUT24)
- net N6_3: now also IC4.21 (HVOUT31); no longer IC4.15 (HVOUT25)
- net N6_4: now also IC4.20 (HVOUT30); no longer IC4.16 (HVOUT26)
- net N6_5: now also IC4.19 (HVOUT29); no longer IC4.17 (HVOUT27)
- net N6_7: now also IC4.17 (HVOUT27); no longer IC4.19 (HVOUT29)
- net N6_8: now also IC4.16 (HVOUT26); no longer IC4.20 (HVOUT30)
- net N6_9: now also IC4.15 (HVOUT25); no longer IC4.21 (HVOUT31)
- net at IC2.33 (~{BL}), IC4.33 (~{BL}): now also IC6.5 (F); no longer IC6.10 (C)
- net at IC2.28 (CLK), IC4.28 (CLK): now also IC6.4 (E); no longer IC6.14 (D)
