File: desgin/nixie_alarm_main_board/12V_DC_plug.kicad_sch (KiCad schematic)
At the start: 5 parts, among them J1 PJ-094H-SMT-TR

Commit message: fixes added
Connections:
- net GND: now also J1.MP1, J1.MP2
Other:
- moved on the sheet: C20, C21, C22, D4, J1
